File: X14-Distribution.brd (EAGLE design)
At the start: 152.4 x 76.2 mm, 57 parts, among them Q1 310mA/60V/1.6Ω, Q2 IRF1018EPBF, Q3 IRF1018EPBF, Q4 IRF1018EPBF, Q5 IRLML5203, Q6 IRLML5203, Q7 IRLML5203, Q8 IRLML5203, U1 DIST_OR_CONTROL_ALTMK06A-M, U2 DIST_OR_CONTROL_ALTMK06A-M

Commit message: Changed a lot of stuff on the board
Parts:
- moved 12V_B_TEST 131.1 mm to (3.78, 16.4)
- moved R8 43.2 mm to (76.2, 49.5), flipped to the top, turned to 0 degrees
- moved Q7 43.2 mm to (78.7, 47.0)
- moved D10 40.6 mm to (74.0, 52.2)
- moved U2 39.4 mm to (71.1, 44.5)
- moved D14 39.4 mm to (68.5, 45.6)
- moved Q4 39.4 mm to (69.8, 33.0)
- moved R9 37.0 mm to (67.0, 49.9), flipped to the top
- moved D8 36.8 mm to (63.9, 43.2)
- moved R5 35.9 mm to (60.6, 44.1), flipped to the top
- moved Q8 35.7 mm to (64.3, 45.9)
- moved BACKPLANE_POWER 24.1 mm to (76.2, 0.00)
- moved BACKPLANE 21.6 mm to (121.6, 5.36)
- moved R10 15.4 mm to (129.2, 14.3), turned to 90 degrees
- moved R11 13.3 mm to (126.8, 12.7), turned to 90 degrees
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Routing:
- net +12V_CONV: track 0.00 -> 153.1 mm, vias 0 -> 2
- net ON/OFF: track 0.00 -> 94.9 mm, vias 0 -> 1
- net D_GND: track 0.00 -> 59.8 mm, vias 0 -> 1
- net +3.3V: track 2.54 -> 57.9 mm
- net 12V_GND: track 5.29 -> 48.4 mm, vias 3 -> 7
- net +12V: track 18.7 -> 47.3 mm, vias 2 -> 4
- net C2_1: track 0.00 -> 28.5 mm, vias 0 -> 2
- net +5V: track 0.00 -> 26.6 mm
- net +12V_A: track 0.00 -> 17.0 mm
- net OR_DRIVE_B: track 11.1 -> 0.00 mm
- net +12V_B: track 22.2 -> 12.0 mm, vias 2 -> 1
- net ALERT_2: track 0.00 -> 7.03 mm
- net DATA: track 0.04 -> 6.86 mm
- net LED_DRIVE_B: track 6.38 -> 0.00 mm, vias 2 -> 0
- net CLK: track 0.00 -> 5.41 mm
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- added copper zone on layer 1, net +48V
- added copper zone on layer 16, net 48V_GND

Commit message: More board stuff
Routing:
- net OR_DRIVE_B: track 0.00 -> 12.8 mm, vias 0 -> 2
- net LED_DRIVE_B: track 0.00 -> 12.7 mm, vias 0 -> 4
- net N$11: track 0.89 -> 6.45 mm
- net N$7: track 0.00 -> 2.67 mm
- net N$15: track 0.00 -> 2.52 mm
- net +12V: track 47.3 -> 49.7 mm

Commit message: Made more changes to the board
Parts:
- moved 12V_B_TEST 131.6 mm to (135.1, 7.65)
- moved D7 13.8 mm to (89.4, 43.6), turned to 180 degrees
- moved R6 12.0 mm to (97.8, 49.5)
- moved D13 11.3 mm to (93.4, 45.5), flipped to the bottom
- moved R4 9.92 mm to (85.1, 44.5), turned to 270 degrees
- moved Q5 9.16 mm to (100.3, 47.0)
- moved Q6 9.05 mm to (89.3, 46.8), turned to 270 degrees
- moved D9 7.41 mm to (95.2, 52.1), turned to 180 degrees
- moved R7 6.94 mm to (92.0, 49.8)
- moved Q3 5.24 mm to (95.2, 33.0)
- moved BRICKS2 5.08 mm to (52.1, 36.8)
- moved D12 4.02 mm to (61.0, 34.3)
- moved U1 3.85 mm to (96.1, 44.5), turned to 270 degrees
- moved 48V_TEST 0.43 mm to (135.1, 2.62)
- moved 12V_TEST 0.42 mm to (135.1, 12.6)
Routing:
- net C2_2: track 0.00 -> 76.1 mm, vias 0 -> 3
- net 48V_GND: track 2.69 -> 73.8 mm, vias 2 -> 4
- net +48V: track 5.73 -> 73.7 mm, vias 2 -> 3
- net +12V_A: track 17.0 -> 58.9 mm, vias 0 -> 3
- net +12V: track 49.7 -> 78.5 mm, vias 4 -> 6
- net OR_DRIVE_A: track 0.00 -> 13.0 mm, vias 0 -> 2
- net LED_DRIVE_A: track 0.00 -> 7.72 mm
- net N$2: track 3.71 -> 11.1 mm
- net N$5: track 0.00 -> 5.75 mm
- net ON/OFF: track 94.9 -> 89.8 mm
- net 12V_GND: track 48.4 -> 52.3 mm, vias 7 -> 12
- net N$13: track 0.00 -> 3.43 mm
- net N$3: track 0.00 -> 3.31 mm
- net +12V_CONV: track 153.1 -> 150.2 mm
- net +12V_B: track 12.0 -> 12.8 mm
- added copper zone on layer 1, net +12V_A

Commit message: Moved the ON/OFF circuit
Parts:
- moved D2 75.1 mm to (19.4, 46.9)
- moved D3 75.1 mm to (14.0, 44.8)
- moved D4 75.1 mm to (20.4, 42.2)
- moved D6 75.1 mm to (24.9, 39.1)
- moved JP1 75.1 mm to (24.8, 43.7)
- moved ON/OFF_TEST 75.1 mm to (30.8, 46.2)
- moved Q1 75.1 mm to (24.8, 36.4)
- moved R2 75.1 mm to (23.8, 46.8)
- moved R3 75.1 mm to (24.5, 41.9)
- moved D5 75.1 mm to (16.1, 39.8)
Routing:
- net ON/OFF: track 89.8 -> 119.8 mm, vias 1 -> 3

Commit message: made some more changes
Routing:
- net ON/OFF: track 119.8 -> 120.3 mm, vias 3 -> 5
Changed lines of the file:
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@@
 <vertex x="33.02" y="34.29"/>
 </polygon>
-<wire x1="109.54" y1="36.83" x2="89.06" y2="57.31" width="0.2032" layer="1"/>
 <via x="31.75" y="36.83" extent="1-16" drill="0.35"/>
-<wire x1="89.06" y1="57.31" x2="89.05194375" y2="57.31805625" width="0.2032" layer="1"/>
-<wire x1="47.4334" y1="48.49840625" x2="46.1634" y2="47.22840625" width="0.2032" layer="16"/>
+<wire x1="67.47" y1="57.31" x2="67.46194375" y2="57.31805625" width="0.2032" layer="1"/>
 <wire x1="46.04" y1="36.83" x2="39.69" y2="30.48" width="0.2032" layer="1"/>
 <wire x1="39.69" y1="30.48" x2="38.1" y2="30.48" width="0.2032" layer="1"/>
@@
 <wire x1="44.45" y1="49.53" x2="44.45" y2="55.88" width="0.2032" layer="1"/>
 <via x="44.45" y="55.88" extent="1-16" drill="0.35"/>
-<wire x1="89.027" y1="57.277" x2="45.847" y2="57.277" width="0.2032" layer="16"/>
+<wire x1="66.167" y1="57.277" x2="45.847" y2="57.277" width="0.2032" layer="16"/>
 <wire x1="44.45" y1="55.88" x2="45.847" y2="57.277" width="0.2032" layer="16"/>
-<wire x1="89.027" y1="57.277" x2="89.06" y2="57.31" width="0.2032" layer="16"/>
-<via x="89.06" y="57.31" extent="1-16" drill="0.35"/>
-<wire x1="44.45" y1="55.88" x2="47.4334" y2="48.49840625" width="0" layer="19" extent="16-16"/>
+<wire x1="66.2" y1="57.31" x2="66.167" y2="57.277" width="0.2032" layer="16"/>
+<wire x1="66.2" y1="57.31" x2="67.47" y2="57.31" width="0.2032" layer="16"/>
+<via x="67.47" y="57.31" extent="1-16" drill="0.35"/>
+<via x="92.71" y="53.34" extent="1-16" drill="0.35"/>
+<wire x1="67.47" y1="57.31" x2="69.8731125" y2="57.31" width="0.2032" layer="1"/>
+<wire x1="69.8731125" y1="57.31" x2="69.9665125" y2="57.4034" width="0.2032" layer="1"/>
+<wire x1="69.9665125" y1="57.4034" x2="88.6466" y2="57.4034" width="0.2032" layer="1"/>
+<wire x1="88.6466" y1="57.4034" x2="92.71" y2="53.34" width="0.2032" layer="1"/>
+<wire x1="92.71" y1="53.34" x2="104.14" y2="41.91" width="0.2032" layer="16"/>
+<via x="104.14" y="41.91" extent="1-16" drill="0.35"/>
+<wire x1="104.14" y1="41.91" x2="104.14" y2="38.1" width="0.2032" layer="1"/>
+<wire x1="104.14" y1="38.1" x2="105.41" y2="36.83" width="0.2032" layer="1"/>
+<wire x1="105.41" y1="36.83" x2="109.54" y2="36.83" width="0.2032" layer="1"/>
 </signal>
 <signal name="GND_RAW">
@@
 <wire x1="74.8042" y1="41.9862" x2="74.9046" y2="41.9862" width="0.4064" layer="1"/>
 <via x="74.9046" y="41.9862" extent="1-16" drill="0.35"/>
-<wire x1="74.9046" y1="41.9862" x2="77.7494" y2="44.831" width="0.4064" layer="16"/>
-<wire x1="77.7494" y1="44.831" x2="77.7494" y2="44.8564" width="0.4064" layer="16"/>
-<via x="77.7494" y="44.8564" extent="1-16" drill="0.35"/>
-<wire x1="77.7494" y1="44.8564" x2="77.7494" y2="45.8494" width="0.4064" layer="1"/>
-<wire x1="77.7494" y1="45.8494" x2="77.79" y2="45.89" width="0.4064" layer="1"/>
+<wire x1="74.9046" y1="41.9862" x2="77.4954" y2="44.577" width="0.4064" layer="16"/>
+<wire x1="77.79" y1="45.89" x2="77.7494" y2="45.8494" width="0.4064" layer="1"/>
+<wire x1="77.79" y1="45.89" x2="77.79" y2="44.8716" width="0.4064" layer="1"/>
+<wire x1="77.79" y1="44.8716" x2="77.4954" y2="44.577" width="0.4064" layer="1"/>
+<via x="77.4954" y="44.577" extent="1-16" drill="0.35"/>
 </signal>
 <signal name="+12V_B">
